File: projects/sensor_data_logger/electronics/generated/kicad/sensor_data_logger.kicad_pcb (KiCad board)
At the start: 2 copper layers, 70 x 50 mm, 16 parts, among them J1 USB-C POWER, J2 UART DEBUG, U1 ESP32-S3-WROOM-1, U2 ICM-42688-P, U3 3V3 Buck

Commit message: fix: sensor_data_logger autorouting pass; add BLE supplier records
- sensor_data_logger: freerouting run to completion, 0 unrouted (routing.json status=pass)
- parts/suppliers/curated.yaml: add nRF52840, BQ24079, BQ27441, JST PH 2-pin,
  SHT31 records for BLE sensor node to resolve supplier_record_missing failures
Parts:
- removed ? (x4): , MountingHole:MountingHole_3.2mm_Pad
- added F1: 500mA Fuse, MIDI, F.Cu at (26.0, 4.00)
- added H1: MountingHole, MountingHole:MountingHole_3.2mm_Pad, F.Cu at (4.00, 4.00)
- added H2: MountingHole, MountingHole:MountingHole_3.2mm_Pad, F.Cu at (66.0, 4.00)
- added H3: MountingHole, MountingHole:MountingHole_3.2mm_Pad, F.Cu at (4.00, 46.0)
- added H4: MountingHole, MountingHole:MountingHole_3.2mm_Pad, F.Cu at (66.0, 46.0)
- added Q1: Ideal Diode, SOT23-6, F.Cu at (34.0, 4.00)
- C1, C2: footprint Capacitor_SMD:C_0603_1608Metric -> C0603
- C9: footprint Capacitor_SMD:C_1206_3216Metric -> C1206
- D1: footprint Package_TO_SOT_SMD:SOT-23-6 -> SOT23-6
- J1: footprint Connector_USB:USB_C_GCT_USB4105 -> USB_C_16Pin
- J2: footprint Connector_Samtec:FTSH-105 -> Cortex_Debug_10Pin
- R1, R2, R3: footprint Resistor_SMD:R_0603_1608Metric -> R0603
- U2: footprint Package_LGA:LGA-14 -> LGA14
- U3: footprint Package_DFN_QFN:VQFN-16 -> VQFN16
Connections:
- U3 pad 1: USB_VBUS -> USB_PROT
Routing:
- net V3V3: track 0.00 -> 109.0 mm
- net USB_DP: track 0.00 -> 52.0 mm, vias 0 -> 1
- net I2C_IMU_SCL: track 0.00 -> 50.2 mm
- net IMU_INT: track 0.00 -> 46.2 mm
- net USB_DM: track 0.00 -> 42.5 mm, vias 0 -> 1
- net I2C_IMU_SDA: track 0.00 -> 41.6 mm
- net BOOT: track 0.00 -> 22.4 mm
- net ESP_EN: track 0.00 -> 20.7 mm
- net UART_RX: track 0.00 -> 18.1 mm
- net UART_TX: track 0.00 -> 13.8 mm
- net USB_DM_RAW: track 0.00 -> 12.5 mm
- net USB_PROT: track 0.00 -> 11.3 mm
- net USB_DP_RAW: track 0.00 -> 10.5 mm
- net USB_VBUS: track 0.00 -> 8.60 mm
- net USB_FUSED: track 0.00 -> 6.00 mm
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